Commit message: Rough Build with ROS2 nodes and web3 blockchain spin

File: ros2_ws/src/robot_logging/urdf/skid_steer.urdf.xacro (robot description, xacro)
@@ -24,56 +24,4 @@
     </collision>
   </link>
-    <!-- LiDAR mast -->
-  <link name="lidar_link">
-    <inertial>
-      <origin xyz="0 0 0" rpy="0 0 0"/>
-      <mass value="0.1"/>
-      <inertia ixx="1e-5" iyy="1e-5" izz="1e-5" ixy="0" ixz="0" iyz="0"/>
-    </inertial>
-    <visual>
-      <origin xyz="0 0 ${wheel_r + base_h + 0.05}" rpy="0 0 0"/>
-      <geometry><cylinder radius="0.02" length="0.10"/></geometry>
-      <material name="grey"><color rgba="0.5 0.5 0.5 1"/></material>
-    </visual>
-    <collision>
-      <origin xyz="0 0 ${wheel_r + base_h + 0.05}" rpy="0 0 0"/>
-      <geometry><cylinder radius="0.02" length="0.10"/></geometry>
-    </collision>
-  </link>
-  <joint name="lidar_joint" type="fixed">
-    <parent link="base_link"/>
-    <child link="lidar_link"/>
-    <!-- mount on top of the chassis -->
-    <origin xyz="0 0 ${wheel_r + base_h/2 + 0.05}" rpy="0 0 0"/>
-  </joint>
-<gazebo reference="lidar_link">
-  <sensor name="lidar" type="lidar">
-    <always_on>true</always_on>
-    <update_rate>10</update_rate>
-    <visualize>true</visualize>
-    <topic>scan</topic>
-    <gz_frame_id>lidar_link</gz_frame_id>
-    <ray>
-      <scan>
-        <horizontal>
-          <samples>720</samples>
-          <resolution>1</resolution>
-          <min_angle>-1.5708</min_angle>   <!-- -90 deg -->
-          <max_angle> 1.5708</max_angle>   <!-- +90 deg -->
-        </horizontal>
-      </scan>
-      <range>
-        <min>0.12</min>
-        <max>10.0</max>
-        <resolution>0.01</resolution>
-      </range>
-      <noise>
-        <type>gaussian</type>
-        <mean>0.0</mean>
-        <stddev>0.01</stddev>
-      </noise>
-    </ray>
-  </sensor>
-</gazebo>
   <!-- Wheel macro -->
   <xacro:macro name="wheel" params="name x y">
@@ -128,5 +76,4 @@
   <minDepth>0.001</minDepth><maxVel>0.2</maxVel><slip1>0.0</slip1><slip2>0.0</slip2>
 </gazebo>
-  <!-- 2D LiDAR (GPU-based) publishing a planar scan -->
   <!-- ros2_control: diff drive using left and right wheel pairs -->
   <ros2_control name="GazeboSimSystem" type="system">
@@ -163,3 +110,59 @@
   </plugin>
 </gazebo>
+<!-- GPU LiDAR link -->
+<link name="lidar_link">
+  <inertial>
+    <origin xyz="0 0 0" rpy="0 0 0"/>
+    <mass value="0.1"/>
+    <inertia ixx="0.0001" iyy="0.0001" izz="0.0001" ixy="0" ixz="0" iyz="0"/>
+  </inertial>
+  <visual>
+    <origin xyz="0 0 0" rpy="0 0 0"/>
+    <geometry>
+      <cylinder radius="0.05" length="0.05"/>
+    </geometry>
+    <material name="black"><color rgba="0.1 0.1 0.1 1"/></material>
+  </visual>
+  <collision>
+    <origin xyz="0 0 0" rpy="0 0 0"/>
+    <geometry>
+      <cylinder radius="0.05" length="0.05"/>
+    </geometry>
+  </collision>
+</link>
+<!-- Fixed joint from base to lidar -->
+<joint name="lidar_joint" type="fixed">
+  <parent link="base_link"/>
+  <child link="lidar_link"/>
+  <!-- Position above base by wheel radius + base height + 5 cm -->
+  <origin xyz="0 0 ${wheel_r + base_h + 0.05}" rpy="0 0 0"/>
+</joint>
+<gazebo reference="lidar_link">
+  <sensor name="gpu_lidar" type="gpu_lidar">
+    <pose>0 0 0 0 0 0</pose>
+    <update_rate>20</update_rate>
+    <visualize>true</visualize>
+    <topic>lidar_points</topic>
+    <horizontal>
+      <samples>720</samples>
+      <resolution>1</resolution>
+      <min_angle>-3.14159</min_angle>
+      <max_angle>3.14159</max_angle>
+    </horizontal>
+    <vertical>
+      <samples>1</samples>
+      <resolution>1</resolution>
+      <min_angle>0.0</min_angle>
+      <max_angle>0.0</max_angle>
+    </vertical>
+    <range>
+      <min>0.12</min>
+      <max>12.0</max>
+      <resolution>0.01</resolution>
+    </range>
+    <plugin name="gpu_lidar_plugin" filename="libgz-sim-gpu-lidar-system.so">
+      <topic>/lidar_points</topic>
+    </plugin>
+  </sensor>
+</gazebo>
 </robot>
